File: kicad/GNSS_Firehose.kicad_pcb (KiCad board)
At the start: 4 copper layers, 117.9 x 99.1 mm, 519 parts, among them J1 SMA, J10 HEADER_16, J2 SMA, J3 SMA, J4 SMA, J5 SMA, J6 HEADER_14, J7 L829-1J1T-43, J8 PJ-063BH, Q1 Si2369DS, U1 MAX2112, U10 MAX19505, U11 AT25DF041A, U12 XC6SLX9-2TQG144C, U15 LMK03806, U17 LTC3633, U18 KSZ9031RNX, U19 CDCLVC1102, U2 MAX19505, U20 MIC2090-1YM5, U21 MIC2090-1YM5, U22 MIC2090-1YM5, U3 MGA-68563, U4 MAX2112, U5 MAX19505, U6 MGA-68563, U7 MAX2112, U8 MAX19505, U9 MGA-68563, Y1 25 MHz

Commit message: Updated PCB
Parts:
- removed FB17: 240, footprints:0402
- removed L10: 0.47 uF, footprints:NRS5020
- removed L11: 1 uH, footprints:NRS5020
- removed L3, L5, L7: 47 nH, footprints:0402
- removed R100, R101, R102, R103, R104, R105: 33, footprints:0402
- removed R133: 10, footprints:0603
- removed R137, R138, R139, R140, R141, R142: 1k, footprints:0402
- removed R143, R87: 0, footprints:1210
- removed R144: 10, footprints:0402
- removed R145: 0, footprints:0805
- removed R146, R147, R148, R149, R150, R72, R73, R76, R77, R78: 10k, footprints:0402
- removed R70: 54.9k, footprints:0402
- removed R71: 12.1k, footprints:0402
- removed R74: 162k, footprints:0402
- removed TP10, TP13, TP14, TP15, TP18, TP19, TP20, TP25, TP26, TP9: test_point, footprints:TP_SMT
- removed U17: LTC3633, footprints:UFD28
- removed U19: CDCLVC1102, footprints:TSSOP8W
- removed the VIA** at (142.6, 79.9)
- removed the VIA** at (147.8, 51.6)
- removed the VIA** at (147.5, 52.5)
- removed the VIA** at (146.8, 51.6)
- removed the VIA** at (146.6, 52.5)
- removed the VIA** at (146.0, 51.6)
- removed the VIA** at (145.5, 52.5)
- removed the VIA** at (145.0, 51.6)
- removed the VIA** at (131.2, 53.4)
- removed the VIA** at (131.2, 51.7)
- removed the VIA** at (159.9, 54.2)
- removed the VIA** at (132.1, 91.2)
- removed the VIA** at (158.9, 55.2)
- removed the VIA** at (158.2, 54.2)
- removed the VIA** at (156.4, 54.1)
- removed the VIA** at (156.4, 56.5)
- removed the VIA** at (154.6, 67.2)
- removed the VIA** at (154.6, 68.5)
- removed the VIA** at (155.1, 69.1)
- removed the VIA** at (162.2, 67.2)
- removed the VIA** at (161.1, 67.2)
- removed the VIA** at (161.6, 68.2)
- removed the VIA** at (133.3, 90.2)
- removed the VIA** at (161.0, 69.1)
- removed the VIA** at (169.8, 67.5)
- removed the VIA** at (170.6, 66.6)
- removed the VIA** at (170.7, 58.4)
- removed the VIA** at (169.8, 57.6)
- removed the VIA** at (136.9, 56.7)
- removed the VIA** at (168.9, 58.4)
- removed the VIA** at (135.6, 56.7)
- removed the VIA** at (132.8, 54.2)
- removed the VIA** at (133.7, 55.1)
- removed the VIA** at (132.2, 90.3)
- removed the VIA** at (134.6, 54.2)
- removed the VIA** at (135.1, 55.3)
- removed the VIA** at (125.5, 53.5)
- removed the VIA** at (124.5, 53.5)
- removed the VIA** at (125.6, 51.6)
- removed the VIA** at (124.5, 51.6)
- removed the VIA** at (162.2, 60.2)
- removed the VIA** at (169.0, 66.8)
- removed the VIA** at (162.2, 69.1)
- removed the VIA** at (155.1, 67.8)
- removed the VIA** at (143.2, 79.2)
- removed the VIA** at (157.2, 55.1)
- removed the VIA** at (144.6, 52.5)
- removed the VIA** at (135.9, 54.4)
- removed the VIA** at (131.2, 52.5)
- removed the VIA** at (125.0, 52.6)
- removed the VIA** at (142.6, 78.4)
- removed the VIA** at (133.9, 91.5)
- removed the VIA** at (141.8, 79.2)
- removed the VIA** at (143.2, 77.7)
- removed the VIA** at (141.9, 77.7)
- removed the VIA** at (148.4, 52.5)
- added C101: 100n, footprints:0402, B.Cu at (144.6, 85.6)
- added C136: 100n, footprints:0402, B.Cu at (140.1, 84.9)
- added C169: 100n, footprints:0402, B.Cu at (138.0, 87.6)
- added C170: 100n, footprints:0402, B.Cu at (139.7, 86.9)
- added C171: 100n, footprints:0402, B.Cu at (133.9, 73.9)
- added C172: 100n, footprints:0402, B.Cu at (128.7, 76.6)
- added C173: 100n, footprints:0402, F.Cu at (121.2, 82.3)
- added C174: 100nF, footprints:0402, F.Cu at (171.8, 63.0)
- added C175: 10uF, footprints:0805, F.Cu at (143.1, 54.7)
- added C178: 10uF, footprints:0805, F.Cu at (156.5, 60.3)
- added C179: 10uF, footprints:0805, F.Cu at (157.4, 65.1)
- added C180: C, footprints:0402, F.Cu at (151.8, 65.0)
- added C181: C, footprints:0402, F.Cu at (156.6, 54.6)
- added C188: C, footprints:0402, F.Cu at (143.2, 48.9)
- added C189: 10uF, footprints:0805, F.Cu at (156.1, 68.2)
- added C190: 10uF, footprints:0805, F.Cu at (153.3, 58.9)
- added C191: 10uF, footprints:0805, F.Cu at (140.0, 53.3)
- added C192: 10uF, footprints:0805, F.Cu at (156.1, 70.3)
- added C2: 100n, footprints:0402, B.Cu at (137.9, 81.1)
- added C256: DNF, footprints:0402, F.Cu at (119.5, 130.2)
- added C257: 100n, footprints:0402, F.Cu at (141.6, 73.6)
- added C258: NONE, footprints:0603, F.Cu at (180.6, 127.6)
- added C3: 100n, footprints:0402, B.Cu at (133.1, 83.5)
- added C38: 100n, footprints:0402, B.Cu at (141.2, 88.9)
- added C39: 100n, footprints:0402, B.Cu at (134.9, 86.7)
- added C4: 100n, footprints:0402, B.Cu at (141.2, 81.9)
- added C40: 100n, footprints:0402, B.Cu at (135.9, 79.8)
- added C48: 100n, footprints:0402, B.Cu at (143.7, 83.6)
- added C50: 100n, footprints:0402, B.Cu at (137.6, 84.1)
- added C52: 100n, footprints:0402, B.Cu at (139.3, 83.3)
- added FB18: L, footprints:0603, F.Cu at (171.2, 64.8)
- added FB19: L, footprints:0603, F.Cu at (134.5, 50.9)
- added J9: HEADER_6, footprints:HEADER6_100MIL, F.Cu at (133.4, 68.2)
- added R12: 33, footprints:0402, F.Cu at (119.5, 69.9)
- added R14: 33, footprints:0402, F.Cu at (119.7, 85.4)
- added R16: 33, footprints:0402, F.Cu at (119.5, 98.8)
- added R24: 330, footprints:0402, F.Cu at (187.7, 93.5)
- added R32: 330, footprints:0402, F.Cu at (187.8, 99.4)
- added R53: 1k, footprints:0402, F.Cu at (122.6, 83.7)
- added R54: 1k, footprints:0402, F.Cu at (122.5, 84.7)
- added R55: 10k, footprints:0402, B.Cu at (133.4, 75.1)
- added R56: 10k, footprints:0402, B.Cu at (128.7, 78.5)
- added R57: 10k, footprints:0402, F.Cu at (122.6, 82.7)
- added R58: 1k, footprints:0402, B.Cu at (143.2, 75.0)
- added R59: 10k, footprints:0402, F.Cu at (142.7, 73.6)
- added R60: NONE, footprints:0603, F.Cu at (180.6, 129.2)
- added R61: R, footprints:0402, F.Cu at (150.7, 63.0)
- added R62: R, footprints:0402, F.Cu at (158.6, 53.6)
- added R63: R, footprints:0402, F.Cu at (145.2, 47.9)
- added R64: R, footprints:0402, F.Cu at (150.7, 65.0)
- added R65: R, footprints:0402, F.Cu at (156.6, 53.6)
- added R66: R, footprints:0402, F.Cu at (143.2, 47.9)
- added R67: 0, footprints:0402, F.Cu at (153.2, 73.0)
- added R68: 0, footprints:0402, F.Cu at (147.5, 58.0)
- added R69: 0, footprints:0402, F.Cu at (164.6, 63.4)
- added R8: 33, footprints:0402, F.Cu at (119.5, 53.8)
- added RN1: 33, footprints:1206_4R, F.Cu at (148.9, 89.6)
- added RN10: 33, footprints:1206_4R, F.Cu at (119.1, 91.9)
- added RN11: 33, footprints:1206_4R, F.Cu at (119.1, 88.0)
- added RN12: 33, footprints:1206_4R, F.Cu at (119.1, 105.4)
- added RN13: 33, footprints:1206_4R, F.Cu at (119.1, 101.3)
- added RN2: 33, footprints:1206_4R, F.Cu at (148.9, 93.5)
- added RN3: 33, footprints:1206_4R, F.Cu at (150.6, 103.3)
- added RN4: 33, footprints:1206_4R, F.Cu at (153.3, 100.7)
- added RN5: 33, footprints:1206_4R, B.Cu at (146.9, 88.7)
- added RN6: 33, footprints:1206_4R, F.Cu at (119.1, 59.9)
- added RN7: 33, footprints:1206_4R, F.Cu at (119.1, 56.0)
- added RN8: 33, footprints:1206_4R, F.Cu at (119.1, 76.1)
- added RN9: 33, footprints:1206_4R, F.Cu at (119.1, 72.2)
- added SW1: Push_SW, footprints:EVQP7, F.Cu at (189.1, 85.2)
- added TP21: test_point, footprints:TP_SMT, F.Cu at (151.7, 63.5)
- added U13: LMZ10501, footprints:LDFN8, F.Cu at (154.2, 64.8)
- added U14: LMZ10501, footprints:LDFN8, F.Cu at (156.8, 57.0)
- added U16: LMZ10501, footprints:LDFN8, F.Cu at (143.4, 51.4)
- added VIA**: , footprints:via_12mil, F.Cu at (155.2, 99.0)
- added VIA**: , footprints:via_12mil, F.Cu at (149.2, 128.6)
- added VIA**: , footprints:via_12mil, F.Cu at (152.0, 97.2)
- added VIA**: , footprints:via_12mil, F.Cu at (151.6, 97.6)
- added VIA**: , footprints:via_12mil, F.Cu at (152.0, 98.1)
- added VIA**: via_12mil, footprints:via_12mil, F.Cu at (146.3, 57.6)
- added VIA**: via_12mil, footprints:via_12mil, F.Cu at (128.9, 51.1)
- added VIA**: via_12mil, footprints:via_12mil, F.Cu at (152.0, 73.0)
- added VIA**: via_12mil, footprints:via_12mil, F.Cu at (156.3, 58.9)
- added VIA**: via_12mil, footprints:via_12mil, F.Cu at (153.9, 67.1)
- added VIA**: via_12mil, footprints:via_12mil, F.Cu at (154.1, 66.3)
- added VIA**: via_12mil, footprints:via_12mil, F.Cu at (153.5, 62.7)
- added VIA**: , footprints:via_12mil, F.Cu at (190.4, 125.3)
- added VIA**: via_12mil, footprints:via_12mil, F.Cu at (154.1, 63.4)
- added VIA**: via_12mil, footprints:via_12mil, F.Cu at (157.1, 67.1)
- added VIA**: via_12mil, footprints:via_12mil, F.Cu at (156.1, 66.4)
- added VIA**: via_12mil, footprints:via_12mil, F.Cu at (156.1, 65.5)
- added VIA**: via_12mil, footprints:via_12mil, F.Cu at (155.3, 58.9)
- added VIA**: via_12mil, footprints:via_12mil, F.Cu at (142.8, 53.3)
- added VIA**: via_12mil, footprints:via_12mil, F.Cu at (154.4, 56.5)
- added VIA**: via_12mil, footprints:via_12mil, F.Cu at (154.5, 59.7)
- added VIA**: via_12mil, footprints:via_12mil, F.Cu at (155.4, 57.0)
- added VIA**: via_12mil, footprints:via_12mil, F.Cu at (158.9, 56.2)
- added VIA**: , footprints:via_12mil, F.Cu at (190.5, 137.8)
- added VIA**: via_12mil, footprints:via_12mil, F.Cu at (158.2, 57.0)
- added VIA**: via_12mil, footprints:via_12mil, F.Cu at (141.1, 50.9)
- added VIA**: via_12mil, footprints:via_12mil, F.Cu at (142.0, 51.4)
- added VIA**: via_12mil, footprints:via_12mil, F.Cu at (155.2, 56.1)
- added VIA**: via_12mil, footprints:via_12mil, F.Cu at (141.9, 50.4)
- added VIA**: via_12mil, footprints:via_12mil, F.Cu at (145.4, 50.5)
- added VIA**: via_12mil, footprints:via_12mil, F.Cu at (144.8, 51.4)
- added VIA**: via_12mil, footprints:via_12mil, F.Cu at (141.9, 53.3)
- added VIA**: via_12mil, footprints:via_12mil, F.Cu at (141.1, 54.2)
- added VIA**: via_12mil, footprints:via_12mil, F.Cu at (153.2, 66.3)
- added VIA**: , footprints:via_12mil, F.Cu at (171.1, 137.8)
- added VIA**: via_12mil, footprints:via_12mil, F.Cu at (151.4, 73.0)
- added VIA**: via_12mil, footprints:via_12mil, F.Cu at (152.0, 73.6)
- added VIA**: via_12mil, footprints:via_12mil, F.Cu at (151.4, 73.6)
- added VIA**: via_12mil, footprints:via_12mil, F.Cu at (128.9, 50.5)
- added VIA**: via_12mil, footprints:via_12mil, F.Cu at (128.3, 50.5)
- added VIA**: via_12mil, footprints:via_12mil, F.Cu at (128.3, 51.1)
- added VIA**: via_12mil, footprints:via_12mil, F.Cu at (146.3, 58.3)
- added VIA**: via_12mil, footprints:via_12mil, F.Cu at (145.6, 58.3)
- added VIA**: via_12mil, footprints:via_12mil, F.Cu at (145.6, 57.6)
- added VIA**: , footprints:via_12mil, F.Cu at (152.5, 97.6)
- added VIA**: , footprints:via_12mil, F.Cu at (160.0, 137.7)
- added VIA**: , footprints:via_12mil, F.Cu at (154.7, 102.5)
- added VIA**: , footprints:via_12mil, F.Cu at (94.3, 62.4)
- added VIA**: , footprints:via_12mil, F.Cu at (103.7, 57.7)
- added VIA**: , footprints:via_12mil, F.Cu at (103.7, 56.9)
- added VIA**: , footprints:via_12mil, F.Cu at (104.6, 56.1)
- added VIA**: , footprints:via_12mil, F.Cu at (106.8, 54.4)
- added VIA**: , footprints:via_12mil, F.Cu at (104.7, 65.2)
- added VIA**: , footprints:via_12mil, F.Cu at (106.3, 66.3)
- added VIA**: , footprints:via_12mil, F.Cu at (99.9, 67.4)
- added VIA**: , footprints:via_12mil, F.Cu at (92.6, 65.3)
- added VIA**: , footprints:via_12mil, F.Cu at (149.8, 137.7)
- added VIA**: , footprints:via_12mil, F.Cu at (126.9, 82.4)
- added VIA**: , footprints:via_12mil, F.Cu at (115.7, 90.7)
- added VIA**: , footprints:via_12mil, F.Cu at (116.5, 105.8)
- added VIA**: , footprints:via_12mil, F.Cu at (107.7, 71.2)
- added VIA**: , footprints:via_12mil, F.Cu at (104.5, 71.9)
- added VIA**: , footprints:via_12mil, F.Cu at (103.7, 72.8)
- added VIA**: , footprints:via_12mil, F.Cu at (103.7, 73.7)
- added VIA**: , footprints:via_12mil, F.Cu at (96.7, 74.4)
- added VIA**: , footprints:via_12mil, F.Cu at (94.3, 73.2)
- added VIA**: , footprints:via_12mil, F.Cu at (93.5, 74.1)
- added VIA**: , footprints:via_12mil, F.Cu at (190.3, 47.6)
- added VIA**: , footprints:via_12mil, F.Cu at (92.3, 73.7)
- added VIA**: , footprints:via_12mil, F.Cu at (91.5, 74.5)
- added VIA**: , footprints:via_12mil, F.Cu at (86.1, 76.1)
- added VIA**: , footprints:via_12mil, F.Cu at (86.1, 75.4)
- added VIA**: , footprints:via_12mil, F.Cu at (87.1, 74.7)
- added VIA**: , footprints:via_12mil, F.Cu at (88.0, 75.4)
- added VIA**: , footprints:via_12mil, F.Cu at (88.0, 76.1)
- added VIA**: , footprints:via_12mil, F.Cu at (89.9, 76.2)
- added VIA**: , footprints:via_12mil, F.Cu at (89.9, 76.9)
- added VIA**: , footprints:via_12mil, F.Cu at (94.4, 78.4)
- added VIA**: , footprints:via_12mil, F.Cu at (172.7, 66.0)
- added VIA**: , footprints:via_12mil, F.Cu at (93.6, 78.5)
- added VIA**: , footprints:via_12mil, F.Cu at (94.3, 79.9)
- added VIA**: , footprints:via_12mil, F.Cu at (95.1, 80.9)
- added VIA**: , footprints:via_12mil, F.Cu at (96.1, 81.7)
- added VIA**: , footprints:via_12mil, F.Cu at (96.2, 82.6)
- added VIA**: , footprints:via_12mil, F.Cu at (97.1, 83.8)
- added VIA**: , footprints:via_12mil, F.Cu at (99.7, 83.8)
- added VIA**: , footprints:via_12mil, F.Cu at (100.5, 82.6)
- added VIA**: , footprints:via_12mil, F.Cu at (99.7, 81.8)
- added VIA**: , footprints:via_12mil, F.Cu at (101.7, 79.4)
- added VIA**: , footprints:via_12mil, F.Cu at (165.4, 65.6)
- added VIA**: , footprints:via_12mil, F.Cu at (102.4, 80.0)
- added VIA**: , footprints:via_12mil, F.Cu at (87.1, 77.9)
- added VIA**: , footprints:via_12mil, F.Cu at (84.4, 77.6)
- added VIA**: , footprints:via_12mil, F.Cu at (83.5, 78.5)
- added VIA**: , footprints:via_12mil, F.Cu at (82.7, 77.6)
- added VIA**: , footprints:via_12mil, F.Cu at (81.3, 77.6)
- added VIA**: , footprints:via_12mil, F.Cu at (78.4, 77.6)
- added VIA**: , footprints:via_12mil, F.Cu at (78.4, 75.9)
- added VIA**: , footprints:via_12mil, F.Cu at (81.2, 75.8)
- added VIA**: , footprints:via_12mil, F.Cu at (83.5, 75.8)
- added VIA**: , footprints:via_12mil, F.Cu at (159.4, 65.1)
- added VIA**: , footprints:via_12mil, F.Cu at (84.0, 75.0)
- added VIA**: , footprints:via_12mil, F.Cu at (111.4, 97.4)
- added VIA**: , footprints:via_12mil, F.Cu at (113.7, 96.3)
- added VIA**: , footprints:via_12mil, F.Cu at (112.9, 98.3)
- added VIA**: , footprints:via_12mil, F.Cu at (111.1, 100.1)
- added VIA**: , footprints:via_12mil, F.Cu at (109.4, 98.9)
- added VIA**: , footprints:via_12mil, F.Cu at (109.5, 101.7)
- added VIA**: , footprints:via_12mil, F.Cu at (107.8, 103.3)
- added VIA**: , footprints:via_12mil, F.Cu at (107.8, 98.7)
- added VIA**: , footprints:via_12mil, F.Cu at (106.1, 98.1)
- added VIA**: , footprints:via_12mil, F.Cu at (163.7, 102.1)
- added VIA**: , footprints:via_12mil, F.Cu at (169.7, 62.9)
- added VIA**: , footprints:via_12mil, F.Cu at (104.7, 97.1)
- added VIA**: , footprints:via_12mil, F.Cu at (103.9, 95.3)
- added VIA**: , footprints:via_12mil, F.Cu at (102.5, 96.4)
- added VIA**: , footprints:via_12mil, F.Cu at (100.0, 98.1)
- added VIA**: , footprints:via_12mil, F.Cu at (100.8, 99.2)
- added VIA**: , footprints:via_12mil, F.Cu at (99.8, 99.8)
- added VIA**: , footprints:via_12mil, F.Cu at (97.2, 99.8)
- added VIA**: , footprints:via_12mil, F.Cu at (96.4, 99.0)
- added VIA**: , footprints:via_12mil, F.Cu at (96.3, 97.9)
- added VIA**: , footprints:via_12mil, F.Cu at (95.1, 97.1)
- added VIA**: , footprints:via_12mil, F.Cu at (174.9, 62.0)
- added VIA**: , footprints:via_12mil, F.Cu at (94.2, 96.0)
- added VIA**: , footprints:via_12mil, F.Cu at (93.4, 94.5)
- added VIA**: , footprints:via_12mil, F.Cu at (94.2, 94.5)
- added VIA**: , footprints:via_12mil, F.Cu at (93.4, 96.4)
- added VIA**: , footprints:via_12mil, F.Cu at (89.9, 92.2)
- added VIA**: , footprints:via_12mil, F.Cu at (90.7, 95.0)
- added VIA**: , footprints:via_12mil, F.Cu at (92.1, 93.2)
- added VIA**: , footprints:via_12mil, F.Cu at (88.0, 92.1)
- added VIA**: , footprints:via_12mil, F.Cu at (88.0, 91.4)
- added VIA**: , footprints:via_12mil, F.Cu at (87.1, 90.7)
- added VIA**: , footprints:via_12mil, F.Cu at (176.7, 60.4)
- added VIA**: , footprints:via_12mil, F.Cu at (86.1, 91.4)
- added VIA**: , footprints:via_12mil, F.Cu at (86.1, 92.0)
- added VIA**: , footprints:via_12mil, F.Cu at (83.5, 91.9)
- added VIA**: , footprints:via_12mil, F.Cu at (81.0, 91.9)
- added VIA**: , footprints:via_12mil, F.Cu at (83.8, 90.9)
- added VIA**: , footprints:via_12mil, F.Cu at (82.6, 93.6)
- added VIA**: , footprints:via_12mil, F.Cu at (83.4, 94.5)
- added VIA**: , footprints:via_12mil, F.Cu at (84.3, 93.6)
- added VIA**: , footprints:via_12mil, F.Cu at (91.2, 90.6)
- added VIA**: , footprints:via_12mil, F.Cu at (92.1, 89.8)
- added VIA**: , footprints:via_12mil, F.Cu at (174.9, 58.7)
- added VIA**: , footprints:via_12mil, F.Cu at (93.5, 90.0)
- added VIA**: , footprints:via_12mil, F.Cu at (94.2, 89.3)
- added VIA**: , footprints:via_12mil, F.Cu at (94.2, 91.9)
- added VIA**: , footprints:via_12mil, F.Cu at (96.7, 90.4)
- added VIA**: , footprints:via_12mil, F.Cu at (103.9, 89.7)
- added VIA**: , footprints:via_12mil, F.Cu at (103.9, 88.7)
- added VIA**: , footprints:via_12mil, F.Cu at (104.7, 87.9)
- added VIA**: , footprints:via_12mil, F.Cu at (106.6, 87.3)
- added VIA**: , footprints:via_12mil, F.Cu at (98.8, 71.7)
- added VIA**: , footprints:via_12mil, F.Cu at (103.9, 96.2)
- added VIA**: , footprints:via_12mil, F.Cu at (173.1, 60.4)
- added VIA**: , footprints:via_12mil, F.Cu at (114.3, 116.8)
- added VIA**: , footprints:via_12mil, F.Cu at (117.4, 119.5)
- added VIA**: , footprints:via_12mil, F.Cu at (162.0, 94.0)
- added VIA**: , footprints:via_12mil, F.Cu at (170.9, 94.0)
- added VIA**: , footprints:via_12mil, F.Cu at (125.4, 65.9)
- added VIA**: , footprints:via_12mil, F.Cu at (124.1, 64.7)
- added VIA**: , footprints:via_12mil, F.Cu at (122.8, 65.9)
- added VIA**: , footprints:via_12mil, F.Cu at (119.8, 78.9)
- added VIA**: , footprints:via_12mil, F.Cu at (120.9, 80.8)
- added VIA**: , footprints:via_12mil, F.Cu at (120.5, 94.2)
- added VIA**: , footprints:via_12mil, F.Cu at (171.8, 61.6)
- added VIA**: , footprints:via_12mil, F.Cu at (123.0, 94.3)
- added VIA**: , footprints:via_12mil, F.Cu at (140.5, 100.3)
- added VIA**: , footprints:via_12mil, F.Cu at (141.7, 101.6)
- added VIA**: , footprints:via_12mil, F.Cu at (131.9, 96.0)
- added VIA**: , footprints:via_12mil, F.Cu at (129.4, 98.6)
- added VIA**: , footprints:via_12mil, F.Cu at (134.1, 93.9)
- added VIA**: , footprints:via_12mil, F.Cu at (126.1, 102.0)
- added VIA**: , footprints:via_12mil, F.Cu at (129.4, 102.8)
- added VIA**: , footprints:via_12mil, F.Cu at (123.6, 104.5)
- added VIA**: , footprints:via_12mil, F.Cu at (125.2, 106.8)
- added VIA**: , footprints:via_12mil, F.Cu at (168.5, 60.7)
- added VIA**: , footprints:via_12mil, F.Cu at (121.3, 110.7)
- added VIA**: , footprints:via_12mil, F.Cu at (114.6, 108.1)
- added VIA**: , footprints:via_12mil, F.Cu at (118.0, 113.7)
- added VIA**: , footprints:via_12mil, F.Cu at (113.3, 113.0)
- added VIA**: , footprints:via_12mil, F.Cu at (110.3, 114.7)
- added VIA**: , footprints:via_12mil, F.Cu at (113.3, 115.0)
- added VIA**: , footprints:via_12mil, F.Cu at (129.4, 105.0)
- added VIA**: , footprints:via_12mil, F.Cu at (128.6, 108.7)
- added VIA**: , footprints:via_12mil, F.Cu at (124.9, 109.6)
- added VIA**: , footprints:via_12mil, F.Cu at (124.4, 112.9)
- added VIA**: , footprints:via_12mil, F.Cu at (165.6, 54.1)
- added VIA**: , footprints:via_12mil, F.Cu at (121.4, 113.0)
- added VIA**: , footprints:via_12mil, F.Cu at (120.5, 117.0)
- added VIA**: , footprints:via_12mil, F.Cu at (117.3, 121.6)
- added VIA**: , footprints:via_12mil, F.Cu at (123.5, 116.2)
- added VIA**: , footprints:via_12mil, F.Cu at (125.5, 113.5)
- added VIA**: , footprints:via_12mil, F.Cu at (132.6, 113.8)
- added VIA**: , footprints:via_12mil, F.Cu at (135.7, 97.5)
- added VIA**: , footprints:via_12mil, F.Cu at (135.7, 102.6)
- added VIA**: , footprints:via_12mil, F.Cu at (135.7, 107.8)
- added VIA**: , footprints:via_12mil, F.Cu at (135.7, 113.6)
- added VIA**: , footprints:via_12mil, F.Cu at (74.5, 47.2)
- added VIA**: , footprints:via_12mil, F.Cu at (135.6, 118.3)
- added VIA**: , footprints:via_12mil, F.Cu at (135.6, 123.4)
- added VIA**: , footprints:via_12mil, F.Cu at (135.6, 128.8)
- added VIA**: , footprints:via_12mil, F.Cu at (135.6, 135.3)
- added VIA**: , footprints:via_12mil, F.Cu at (130.4, 115.6)
- added VIA**: , footprints:via_12mil, F.Cu at (126.7, 119.4)
- added VIA**: , footprints:via_12mil, F.Cu at (123.0, 122.7)
- added VIA**: , footprints:via_12mil, F.Cu at (122.2, 126.3)
- added VIA**: , footprints:via_12mil, F.Cu at (123.4, 125.3)
- added VIA**: , footprints:via_12mil, F.Cu at (120.5, 127.8)
- added VIA**: , footprints:via_12mil, F.Cu at (85.8, 47.0)
- added VIA**: , footprints:via_12mil, F.Cu at (128.8, 125.2)
- added VIA**: , footprints:via_12mil, F.Cu at (131.4, 127.9)
- added VIA**: , footprints:via_12mil, F.Cu at (127.2, 131.3)
- added VIA**: , footprints:via_12mil, F.Cu at (118.4, 127.6)
- added VIA**: , footprints:via_12mil, F.Cu at (118.1, 131.7)
- added VIA**: , footprints:via_12mil, F.Cu at (105.2, 131.6)
- added VIA**: , footprints:via_12mil, F.Cu at (100.2, 119.3)
- added VIA**: , footprints:via_12mil, F.Cu at (99.3, 120.2)
- added VIA**: , footprints:via_12mil, F.Cu at (100.3, 122.6)
- added VIA**: , footprints:via_12mil, F.Cu at (99.4, 123.4)
- added VIA**: , footprints:via_12mil, F.Cu at (119.1, 57.8)
- added VIA**: , footprints:via_12mil, F.Cu at (93.5, 47.1)
- added VIA**: , footprints:via_12mil, F.Cu at (100.3, 126.6)
- added VIA**: , footprints:via_12mil, F.Cu at (99.4, 127.5)
- added VIA**: , footprints:via_12mil, F.Cu at (95.4, 127.5)
- added VIA**: , footprints:via_12mil, F.Cu at (94.5, 126.7)
- added VIA**: , footprints:via_12mil, F.Cu at (95.5, 123.2)
- added VIA**: , footprints:via_12mil, F.Cu at (94.7, 122.3)
- added VIA**: , footprints:via_12mil, F.Cu at (94.6, 119.2)
- added VIA**: , footprints:via_12mil, F.Cu at (104.5, 103.9)
- added VIA**: , footprints:via_12mil, F.Cu at (103.8, 105.4)
- added VIA**: , footprints:via_12mil, F.Cu at (103.8, 106.2)
- added VIA**: , footprints:via_12mil, F.Cu at (100.9, 47.1)
- added VIA**: , footprints:via_12mil, F.Cu at (104.1, 109.3)
- added VIA**: , footprints:via_12mil, F.Cu at (103.8, 111.2)
- added VIA**: , footprints:via_12mil, F.Cu at (103.7, 112.3)
- added VIA**: , footprints:via_12mil, F.Cu at (104.5, 113.6)
- added VIA**: , footprints:via_12mil, F.Cu at (101.5, 111.3)
- added VIA**: , footprints:via_12mil, F.Cu at (100.4, 111.2)
- added VIA**: , footprints:via_12mil, F.Cu at (99.6, 110.3)
- added VIA**: , footprints:via_12mil, F.Cu at (99.7, 107.5)
- added VIA**: , footprints:via_12mil, F.Cu at (100.5, 108.3)
- added VIA**: , footprints:via_12mil, F.Cu at (101.6, 108.4)
- added VIA**: , footprints:via_12mil, F.Cu at (108.2, 47.2)
- added VIA**: , footprints:via_12mil, F.Cu at (95.7, 109.6)
- added VIA**: , footprints:via_12mil, F.Cu at (94.8, 110.4)
- added VIA**: , footprints:via_12mil, F.Cu at (91.8, 109.7)
- added VIA**: , footprints:via_12mil, F.Cu at (90.9, 110.4)
- added VIA**: , footprints:via_12mil, F.Cu at (88.9, 110.5)
- added VIA**: , footprints:via_12mil, F.Cu at (88.0, 109.6)
- added VIA**: , footprints:via_12mil, F.Cu at (86.6, 109.7)
- added VIA**: , footprints:via_12mil, F.Cu at (85.7, 110.4)
- added VIA**: , footprints:via_12mil, F.Cu at (84.9, 109.6)
- added VIA**: , footprints:via_12mil, F.Cu at (88.8, 118.0)
- added VIA**: , footprints:via_12mil, F.Cu at (115.8, 47.1)
- added VIA**: , footprints:via_12mil, F.Cu at (88.0, 118.9)
- added VIA**: , footprints:via_12mil, F.Cu at (88.7, 119.7)
- added VIA**: , footprints:via_12mil, F.Cu at (88.7, 122.0)
- added VIA**: , footprints:via_12mil, F.Cu at (88.0, 122.7)
- added VIA**: , footprints:via_12mil, F.Cu at (88.8, 123.6)
- added VIA**: , footprints:via_12mil, F.Cu at (87.8, 125.6)
- added VIA**: , footprints:via_12mil, F.Cu at (87.0, 126.5)
- added VIA**: , footprints:via_12mil, F.Cu at (86.2, 125.6)
- added VIA**: , footprints:via_12mil, F.Cu at (84.7, 125.6)
- added VIA**: , footprints:via_12mil, F.Cu at (83.9, 126.4)
- added VIA**: , footprints:via_12mil, F.Cu at (123.5, 47.1)
- added VIA**: , footprints:via_12mil, F.Cu at (83.1, 125.6)
- added VIA**: , footprints:via_12mil, F.Cu at (81.3, 109.6)
- added VIA**: , footprints:via_12mil, F.Cu at (81.3, 107.8)
- added VIA**: , footprints:via_12mil, F.Cu at (84.9, 107.8)
- added VIA**: , footprints:via_12mil, F.Cu at (90.9, 107.8)
- added VIA**: , footprints:via_12mil, F.Cu at (95.5, 107.9)
- added VIA**: , footprints:via_12mil, F.Cu at (100.4, 105.8)
- added VIA**: , footprints:via_12mil, F.Cu at (88.8, 114.8)
- added VIA**: , footprints:via_12mil, F.Cu at (93.1, 113.1)
- added VIA**: , footprints:via_12mil, F.Cu at (96.1, 111.4)
- added VIA**: , footprints:via_12mil, F.Cu at (130.4, 47.1)
- added VIA**: , footprints:via_12mil, F.Cu at (96.1, 113.9)
- added VIA**: , footprints:via_12mil, F.Cu at (91.3, 114.8)
- added VIA**: , footprints:via_12mil, F.Cu at (90.6, 119.2)
- added VIA**: , footprints:via_12mil, F.Cu at (90.5, 124.2)
- added VIA**: , footprints:via_12mil, F.Cu at (85.5, 123.8)
- added VIA**: , footprints:via_12mil, F.Cu at (80.4, 123.8)
- added VIA**: , footprints:via_12mil, F.Cu at (80.3, 125.7)
- added VIA**: , footprints:via_12mil, F.Cu at (114.8, 133.1)
- added VIA**: , footprints:via_12mil, F.Cu at (110.7, 133.1)
- added VIA**: , footprints:via_12mil, F.Cu at (107.0, 133.1)
- added VIA**: , footprints:via_12mil, F.Cu at (138.7, 47.3)
- added VIA**: , footprints:via_12mil, F.Cu at (102.9, 133.1)
- added VIA**: , footprints:via_12mil, F.Cu at (98.3, 133.1)
- added VIA**: , footprints:via_12mil, F.Cu at (93.1, 133.0)
- added VIA**: , footprints:via_12mil, F.Cu at (90.6, 130.8)
- added VIA**: , footprints:via_12mil, F.Cu at (90.6, 127.2)
- added VIA**: , footprints:via_12mil, F.Cu at (88.8, 127.2)
- added VIA**: , footprints:via_12mil, F.Cu at (88.7, 131.5)
- added VIA**: , footprints:via_12mil, F.Cu at (91.4, 134.1)
- added VIA**: , footprints:via_12mil, F.Cu at (98.3, 134.8)
- added VIA**: , footprints:via_12mil, F.Cu at (102.9, 134.9)
- added VIA**: , footprints:via_12mil, F.Cu at (147.6, 47.5)
- added VIA**: , footprints:via_12mil, F.Cu at (106.9, 134.9)
- added VIA**: , footprints:via_12mil, F.Cu at (110.7, 134.9)
- added VIA**: , footprints:via_12mil, F.Cu at (114.9, 135.0)
- added VIA**: , footprints:via_12mil, F.Cu at (119.4, 133.3)
- added VIA**: , footprints:via_12mil, F.Cu at (120.6, 131.4)
- added VIA**: , footprints:via_12mil, F.Cu at (123.5, 131.3)
- added VIA**: , footprints:via_12mil, F.Cu at (81.3, 93.6)
- added VIA**: , footprints:via_12mil, F.Cu at (125.1, 93.7)
- added VIA**: , footprints:via_12mil, F.Cu at (114.6, 92.4)
- added VIA**: , footprints:via_12mil, F.Cu at (117.0, 93.8)
- added VIA**: , footprints:via_12mil, F.Cu at (155.8, 47.5)
- added VIA**: , footprints:via_12mil, F.Cu at (118.3, 97.4)
- added VIA**: , footprints:via_12mil, F.Cu at (114.5, 76.4)
- added VIA**: , footprints:via_12mil, F.Cu at (115.9, 74.7)
- added VIA**: , footprints:via_12mil, F.Cu at (117.2, 78.0)
- added VIA**: , footprints:via_12mil, F.Cu at (116.4, 79.5)
- added VIA**: , footprints:via_12mil, F.Cu at (123.8, 80.1)
- added VIA**: , footprints:via_12mil, F.Cu at (118.1, 82.0)
- added VIA**: , footprints:via_12mil, F.Cu at (112.9, 82.0)
- added VIA**: , footprints:via_12mil, F.Cu at (123.6, 70.0)
- added VIA**: , footprints:via_12mil, F.Cu at (113.6, 68.2)
- added VIA**: , footprints:via_12mil, F.Cu at (163.9, 47.6)
- added VIA**: , footprints:via_12mil, F.Cu at (119.2, 68.1)
- added VIA**: , footprints:via_12mil, F.Cu at (121.1, 61.9)
- added VIA**: , footprints:via_12mil, F.Cu at (114.6, 60.4)
- added VIA**: , footprints:via_12mil, F.Cu at (116.4, 63.4)
- added VIA**: , footprints:via_12mil, F.Cu at (111.2, 65.1)
- added VIA**: , footprints:via_12mil, F.Cu at (109.2, 68.2)
- added VIA**: , footprints:via_12mil, F.Cu at (115.9, 58.8)
- added VIA**: , footprints:via_12mil, F.Cu at (128.8, 52.7)
- added VIA**: , footprints:via_12mil, F.Cu at (131.1, 52.7)
- added VIA**: , footprints:via_12mil, F.Cu at (133.5, 52.7)
- added VIA**: , footprints:via_12mil, F.Cu at (118.4, 52.3)
- added VIA**: , footprints:via_12mil, F.Cu at (173.0, 47.6)
- added VIA**: , footprints:via_12mil, F.Cu at (132.2, 53.9)
- added VIA**: , footprints:via_12mil, F.Cu at (130.1, 53.9)
- added VIA**: , footprints:via_12mil, F.Cu at (108.0, 52.3)
- added VIA**: , footprints:via_12mil, F.Cu at (111.8, 52.3)
- added VIA**: , footprints:via_12mil, F.Cu at (114.8, 52.3)
- added VIA**: , footprints:via_12mil, F.Cu at (107.8, 85.0)
- added VIA**: , footprints:via_12mil, F.Cu at (146.8, 86.6)
- added VIA**: , footprints:via_12mil, F.Cu at (149.4, 86.6)
- added VIA**: , footprints:via_12mil, F.Cu at (152.2, 89.2)
- added VIA**: , footprints:via_12mil, F.Cu at (154.8, 91.8)
- added VIA**: , footprints:via_12mil, F.Cu at (148.5, 53.8)
- added VIA**: , footprints:via_12mil, F.Cu at (159.2, 96.2)
- added VIA**: , footprints:via_12mil, F.Cu at (160.3, 99.4)
- added VIA**: , footprints:via_12mil, F.Cu at (140.6, 96.5)
- added VIA**: , footprints:via_12mil, F.Cu at (150.4, 97.0)
- added VIA**: , footprints:via_12mil, F.Cu at (161.6, 111.2)
- added VIA**: , footprints:via_12mil, F.Cu at (159.8, 113.0)
- added VIA**: , footprints:via_12mil, F.Cu at (156.9, 114.9)
- added VIA**: , footprints:via_12mil, F.Cu at (152.2, 115.0)
- added VIA**: , footprints:via_12mil, F.Cu at (149.7, 113.8)
- added VIA**: , footprints:via_12mil, F.Cu at (156.4, 113.4)
- added VIA**: , footprints:via_12mil, F.Cu at (154.8, 52.4)
- added VIA**: , footprints:via_12mil, F.Cu at (172.1, 112.6)
- added VIA**: , footprints:via_12mil, F.Cu at (169.1, 113.7)
- added VIA**: , footprints:via_12mil, F.Cu at (169.1, 110.1)
- added VIA**: , footprints:via_12mil, F.Cu at (172.1, 110.0)
- added VIA**: , footprints:via_12mil, F.Cu at (172.0, 118.7)
- added VIA**: , footprints:via_12mil, F.Cu at (169.6, 121.6)
- added VIA**: , footprints:via_12mil, F.Cu at (171.8, 121.9)
- added VIA**: , footprints:via_12mil, F.Cu at (174.2, 120.8)
- added VIA**: , footprints:via_12mil, F.Cu at (174.3, 114.6)
- added VIA**: , footprints:via_12mil, F.Cu at (174.5, 111.0)
- added VIA**: , footprints:via_12mil, F.Cu at (160.9, 54.1)
- added VIA**: , footprints:via_12mil, F.Cu at (167.2, 120.0)
- added VIA**: , footprints:via_12mil, F.Cu at (162.6, 118.3)
- added VIA**: , footprints:via_12mil, F.Cu at (159.5, 115.2)
- added VIA**: , footprints:via_12mil, F.Cu at (163.5, 110.5)
- added VIA**: , footprints:via_12mil, F.Cu at (166.3, 113.3)
- added VIA**: , footprints:via_12mil, F.Cu at (164.9, 105.0)
- added VIA**: , footprints:via_12mil, F.Cu at (157.7, 101.2)
- added VIA**: , footprints:via_12mil, F.Cu at (157.1, 98.8)
- added VIA**: , footprints:via_12mil, F.Cu at (129.7, 94.7)
- added VIA**: , footprints:via_12mil, F.Cu at (114.7, 103.4)
- added VIA**: , footprints:via_12mil, F.Cu at (158.8, 59.0)
- added VIA**: , footprints:via_12mil, F.Cu at (124.0, 100.3)
- added VIA**: , footprints:via_12mil, F.Cu at (107.7, 68.2)
- added VIA**: , footprints:via_12mil, F.Cu at (109.9, 83.0)
- added VIA**: , footprints:via_12mil, F.Cu at (109.7, 87.9)
- added VIA**: , footprints:via_12mil, F.Cu at (89.8, 79.5)
- added VIA**: , footprints:via_12mil, F.Cu at (87.1, 94.1)
- added VIA**: , footprints:via_12mil, F.Cu at (88.8, 96.0)
- added VIA**: , footprints:via_12mil, F.Cu at (92.8, 67.1)
- added VIA**: , footprints:via_12mil, F.Cu at (89.9, 72.9)
- added VIA**: , footprints:via_12mil, F.Cu at (88.3, 81.5)
- added VIA**: , footprints:via_12mil, F.Cu at (182.3, 129.2)
- added VIA**: , footprints:via_12mil, F.Cu at (89.8, 82.1)
- added VIA**: , footprints:via_12mil, F.Cu at (88.3, 88.3)
- added VIA**: , footprints:via_12mil, F.Cu at (89.8, 88.4)
- added VIA**: , footprints:via_12mil, F.Cu at (91.6, 88.3)
- added VIA**: , footprints:via_12mil, F.Cu at (92.7, 99.2)
- added VIA**: , footprints:via_12mil, F.Cu at (94.6, 103.0)
- added VIA**: , footprints:via_12mil, F.Cu at (94.6, 106.3)
- added VIA**: , footprints:via_12mil, F.Cu at (93.2, 105.4)
- added VIA**: , footprints:via_12mil, F.Cu at (88.7, 105.8)
- added VIA**: , footprints:via_12mil, F.Cu at (87.1, 105.6)
- added VIA**: , footprints:via_12mil, F.Cu at (182.3, 127.5)
- added VIA**: , footprints:via_12mil, F.Cu at (89.7, 113.3)
- added VIA**: , footprints:via_12mil, F.Cu at (92.5, 119.2)
- added VIA**: , footprints:via_12mil, F.Cu at (94.5, 115.6)
- added VIA**: , footprints:via_12mil, F.Cu at (93.3, 116.4)
- added VIA**: , footprints:via_12mil, F.Cu at (189.2, 96.8)
- added VIA**: , footprints:via_12mil, F.Cu at (189.1, 91.0)
- added VIA**: , footprints:via_12mil, F.Cu at (187.3, 87.2)
- added VIA**: , footprints:via_12mil, F.Cu at (189.2, 77.0)
- added VIA**: , footprints:via_12mil, F.Cu at (190.3, 104.5)
- added VIA**: , footprints:via_12mil, F.Cu at (180.1, 101.5)
- added VIA**: , footprints:via_12mil, F.Cu at (181.7, 126.5)
- added VIA**: , footprints:via_12mil, F.Cu at (180.0, 96.3)
- added VIA**: , footprints:via_12mil, F.Cu at (180.1, 88.5)
- added VIA**: , footprints:via_12mil, F.Cu at (180.1, 83.0)
- added VIA**: , footprints:via_12mil, F.Cu at (180.4, 73.5)
- added VIA**: , footprints:via_12mil, F.Cu at (172.2, 73.5)
- added VIA**: , footprints:via_12mil, F.Cu at (172.1, 83.0)
- added VIA**: , footprints:via_12mil, F.Cu at (171.8, 88.9)
- added VIA**: , footprints:via_12mil, F.Cu at (171.1, 102.0)
- added VIA**: , footprints:via_12mil, F.Cu at (174.9, 104.2)
- added VIA**: , footprints:via_12mil, F.Cu at (183.4, 105.7)
- added VIA**: , footprints:via_12mil, F.Cu at (190.8, 85.4)
- added VIA**: , footprints:via_12mil, F.Cu at (162.5, 73.5)
- added VIA**: , footprints:via_12mil, F.Cu at (150.5, 70.9)
- added VIA**: , footprints:via_12mil, F.Cu at (142.1, 70.8)
- added VIA**: , footprints:via_12mil, F.Cu at (139.7, 75.0)
- added VIA**: , footprints:via_12mil, F.Cu at (141.2, 59.1)
- added VIA**: , footprints:via_12mil, F.Cu at (136.3, 57.8)
- added VIA**: , footprints:via_12mil, F.Cu at (128.8, 57.7)
- added VIA**: , footprints:via_12mil, F.Cu at (147.6, 82.8)
- added VIA**: , footprints:via_12mil, F.Cu at (150.0, 81.0)
- added VIA**: , footprints:via_12mil, F.Cu at (156.3, 81.0)
- added VIA**: , footprints:via_12mil, F.Cu at (153.8, 74.0)
- added VIA**: , footprints:via_12mil, F.Cu at (158.2, 85.1)
- added VIA**: , footprints:via_12mil, F.Cu at (158.2, 88.2)
- added VIA**: , footprints:via_12mil, F.Cu at (160.1, 82.8)
- added VIA**: , footprints:via_12mil, F.Cu at (161.9, 82.8)
- added VIA**: , footprints:via_12mil, F.Cu at (162.0, 88.8)
- added VIA**: , footprints:via_12mil, F.Cu at (160.9, 90.7)
- added VIA**: , footprints:via_12mil, F.Cu at (162.4, 76.2)
- added VIA**: , footprints:via_12mil, F.Cu at (137.9, 97.5)
- added VIA**: , footprints:via_12mil, F.Cu at (139.4, 102.6)
- added VIA**: , footprints:via_12mil, F.Cu at (140.2, 113.6)
- added VIA**: , footprints:via_12mil, F.Cu at (98.4, 50.8)
- added VIA**: , footprints:via_12mil, F.Cu at (131.4, 68.3)
- added VIA**: , footprints:via_12mil, F.Cu at (140.0, 118.2)
- added VIA**: , footprints:via_12mil, F.Cu at (139.9, 123.4)
- added VIA**: , footprints:via_12mil, F.Cu at (140.2, 128.9)
- added VIA**: , footprints:via_12mil, F.Cu at (140.1, 135.1)
- added VIA**: , footprints:via_12mil, F.Cu at (140.0, 107.8)
- added VIA**: , footprints:via_12mil, F.Cu at (135.5, 73.5)
- added VIA**: , footprints:via_12mil, F.Cu at (139.6, 66.4)
- added VIA**: , footprints:via_12mil, F.Cu at (137.4, 70.0)
- added VIA**: , footprints:via_12mil, F.Cu at (139.6, 69.9)
- added VIA**: , footprints:via_12mil, F.Cu at (119.9, 118.9)
- added VIA**: , footprints:via_12mil, F.Cu at (119.0, 115.5)
- added VIA**: , footprints:via_12mil, F.Cu at (127.2, 107.4)
- added VIA**: , footprints:via_12mil, F.Cu at (127.8, 104.2)
- added VIA**: , footprints:via_12mil, F.Cu at (127.8, 100.3)
- added VIA**: , footprints:via_12mil, F.Cu at (172.0, 128.5)
- added VIA**: , footprints:via_12mil, F.Cu at (127.8, 96.6)
- added VIA**: , footprints:via_12mil, F.Cu at (120.6, 121.8)
- added VIA**: , footprints:via_12mil, F.Cu at (119.7, 122.2)
- added VIA**: , footprints:via_12mil, F.Cu at (80.1, 56.9)
- added VIA**: , footprints:via_12mil, F.Cu at (79.2, 57.8)
- added VIA**: , footprints:via_12mil, F.Cu at (84.1, 58.7)
- added VIA**: , footprints:via_12mil, F.Cu at (83.5, 59.8)
- added VIA**: , footprints:via_12mil, F.Cu at (80.9, 59.9)
- added VIA**: , footprints:via_12mil, F.Cu at (78.6, 61.6)
- added VIA**: , footprints:via_12mil, F.Cu at (80.9, 61.6)
- added VIA**: , footprints:via_12mil, F.Cu at (159.8, 119.7)
- added VIA**: , footprints:via_12mil, F.Cu at (86.2, 61.5)
- added VIA**: , footprints:via_12mil, F.Cu at (83.4, 62.4)
- added VIA**: , footprints:via_12mil, F.Cu at (84.3, 61.6)
- added VIA**: , footprints:via_12mil, F.Cu at (82.7, 61.6)
- added VIA**: , footprints:via_12mil, F.Cu at (89.9, 61.0)
- added VIA**: , footprints:via_12mil, F.Cu at (89.9, 63.5)
- added VIA**: , footprints:via_12mil, F.Cu at (90.7, 62.8)
- added VIA**: , footprints:via_12mil, F.Cu at (90.7, 61.7)
- added VIA**: , footprints:via_12mil, F.Cu at (89.8, 60.1)
- added VIA**: , footprints:via_12mil, F.Cu at (88.0, 60.1)
- added VIA**: , footprints:via_12mil, F.Cu at (149.0, 119.9)
- added VIA**: , footprints:via_12mil, F.Cu at (88.0, 59.4)
- added VIA**: , footprints:via_12mil, F.Cu at (87.0, 58.7)
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Connections:
- net /RF Channel 2/ch2_gc1_lpf renamed Net-(C81-Pad1)
- net /RF Channel 2/ch2_xtal renamed Net-(C100-Pad2)
- net /RF Channel 3/ch3_gc1_lpf renamed Net-(C116-Pad1)
- net /RF Channel 3/ch3_xtal renamed Net-(C135-Pad2)
- net /RF Channel 4/10_MHz- renamed Net-(C138-Pad2)
- net /RF Channel 4/PPS- renamed Net-(C140-Pad2)
- net /RF channel 1/ch1_gc1_lpf renamed Net-(C18-Pad1)
- C129 pad 1: VCC_3.3V -> VCC_3V3_AN
- C130 pad 1: VCC_3.3V -> VCC_3V3_AN
- C131 pad 1: VCC_3.3V -> VCC_3V3_AN
- C132 pad 1: VCC_3.3V -> VCC_3V3_AN
- C133 pad 1: VCC_3.3V -> VCC_3V3_DIG
- C134 pad 1: VCC_3.3V -> VCC_3V3_DIG
- C147 pad 1: VCC_3.3V -> VCC_3V3_DIG
- C148 pad 1: VCC_3.3V -> VCC_3V3_DIG
- C149 pad 1: VCC_3.3V -> VCC_3V3_DIG
- C150 pad 1: VCC_3.3V -> VCC_3V3_DIG
- C151 pad 1: VCC_3.3V -> VCC_3V3_DIG
- C152 pad 1: VCC_3.3V -> VCC_3V3_DIG
- C153 pad 1: VCC_3.3V -> VCC_3V3_DIG
- C154 pad 1: VCC_3.3V -> VCC_3V3_DIG
- C155 pad 1: VCC_3.3V -> VCC_3V3_DIG
- C156 pad 1: VCC_3.3V -> Net-(C156-Pad1)
- C156 pad 2: GND -> AUX_CLK
- C157 pad 1: VCC_3.3V -> VCC_3V3_DIG
- C158 pad 1: VCC_3.3V -> VCC_3V3_DIG
- C159 pad 1: VCC_3.3V -> VCC_3V3_DIG
- C160 pad 1: VCC_3.3V -> VCC_3V3_DIG
- C161 pad 1: VCC_3.3V -> VCC_3V3_DIG
- C162 pad 1: VCC_3.3V -> VCC_3V3_DIG
- C163 pad 1: VCC_3.3V -> VCC_3V3_DIG
- C164 pad 1: VCC_3.3V -> VCC_3V3_DIG
- C165 pad 1: VCC_3.3V -> VCC_3V3_DIG
- C166 pad 1: VCC_3.3V -> VCC_3V3_DIG
- C167 pad 1: VCC_3.3V -> VCC_3V3_DIG
- C168 pad 1: VCC_3.3V -> VCC_3V3_DIG
- C194 pad 1: Net-(C194-Pad1) -> Net-(C190-Pad1)
- C195 pad 1: Net-(C195-Pad1) -> Net-(C191-Pad1)
- C197 pad 1: Net-(C197-Pad1) -> Net-(C190-Pad1)
- C197 pad 2: Net-(C197-Pad2) -> GND
- C198 pad 1: Net-(C194-Pad1) -> Net-(C191-Pad1)
- C199 pad 1: Net-(C199-Pad1) -> VCC_3V3_AN
- C199 pad 2: Net-(C199-Pad2) -> GND
- C200 pad 1: Net-(C200-Pad1) -> VCC_3V3_AN
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Routing:
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- added copper zone on B.Cu, net /Ethernet/DVDDH
- added copper zone on B.Cu, net /Ethernet/DVDDL
- added copper zone on B.Cu, net GND
- added copper zone on In2.Cu, net GND
- added copper zone on F.Cu, net Net-(C174-Pad1)
- added copper zone on F.Cu, net Net-(C175-Pad1)
- added copper zone on F.Cu, net Net-(C190-Pad1)
- added copper zone on F.Cu, net Net-(C191-Pad1)
- added copper zone on F.Cu, net Net-(FB18-Pad2)
- added copper zone on F.Cu, net VCC_3V3_AN
- added copper zone on In2.Cu, net VCC_3V3_AN
- added copper zone on F.Cu, net VCC_3V3_DIG
- added copper zone on In2.Cu, net VCC_3V3_DIG
- removed copper zone on In1.Cu, net /Ethernet/chassis_gnd
- removed copper zone on In2.Cu, net /RF Channel 2/ch2_vcc_lna
- removed copper zone on In2.Cu, net /RF Channel 3/ch3_vcc_lna
- removed copper zone on In2.Cu, net /RF channel 1/ch1_vcc_lna
- removed copper zone on B.Cu, net Net-(C194-Pad1)
- removed copper zone on F.Cu, net Net-(C194-Pad1)
- removed copper zone on F.Cu, net Net-(C197-Pad1)
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Other:
- board text added: "1"
- board text added: "15"
- board text added: "16"
- board text added: "2"
- board text added: "3V3"
- board text added: "Alan Page April 2018 version 0.1"
- board text added: "GND"
- board text added: "P/N ????-?? REV 0.1"
- board text added: "SOFT RESET"
- board text added: "TCLK"
- board text added: "TDI"
- board text added: "TDO"
- board text added: "TMS"
- board text removed: "1.2 V"
- board text removed: "3.3 V"
- board text removed: "P/N 1002-01 REV 2.2"
- board text removed: "Peter Monta April 2017 version 2.2"
